File: 5.0mustangProteusPnP.kicad_sch (KiCad schematic)
At the start: 5 parts, among them J1 5-146280-3, J2 5103308-3, J4 5103308-3, U1 FORD60PIN

Commit message: add WBO module in sch
Parts:
- added J10, J7: XH-10AW, Connector_JST:JST_XH_S10B-XH-A_1x10_P2.50mm_Horizontal, symbol Connector_Generic:Conn_01x10
- added J13, J3: Conn_01x06, Connector_PinHeader_2.54mm:PinHeader_1x06_P2.54mm_Vertical, symbol Connector_Generic:Conn_01x06
- added M1, M3: Module-wbo-0.3, hellen-one-wbo-0.3:wbo, symbol hellen-one-wbo-0.3:Module-wbo-0.3
- added M2, M4: Module-can-0.1, hellen-one-can-0.1:can, symbol hellen-one-can-0.1:Module-can-0.1
Connections:
- net 12V_MR: now also J10.1 (Pin_1), J10.2 (Pin_2), J7.1 (Pin_1), J7.2 (Pin_2)
- net GND: now also J10.10 (Pin_10), J10.9 (Pin_9), J13.3 (Pin_3), J3.3 (Pin_3), J7.10 (Pin_10), J7.9 (Pin_9), M1.E6 (LSU_H-), M1.G (GND), M2.E1 (GND), M3.E6 (LSU_H-), M3.G (GND), M4.E1 (GND)
- new net: M2.V2 (CAN_VIO), M3.W2 (CAN_VIO)
- new net: M2.V5 (CAN_TX), M3.W4 (CAN_TX)
- new net: M2.V6 (CAN_RX), M3.W3 (CAN_RX)
- new net: J3.1 (Pin_1), M3.W8 (V33_OUT)
- new net: J3.2 (Pin_2), M3.W7 (SWCLK)
- new net: J3.4 (Pin_4), M3.W6 (SWDIO)
- new net: J3.5 (Pin_5), M3.W5 (nReset)
- new net: J10.3 (Pin_3), M3.E1 (LSU_Un)
- new net: J10.4 (Pin_4), M3.E2 (LSU_Vm)
- new net: J10.5 (Pin_5), M3.E3 (LSU_Ip)
- new net: J10.6 (Pin_6), M3.E4 (LSU_Rtrim)
- new net: J10.7 (Pin_7), J10.8 (Pin_8), M3.E5 (LSU_H+)
- new net: M3.J1 (SEL1), M3.J_GND1 (PULL_DOWN1)
- new net: J13.1 (Pin_1), M1.W8 (V33_OUT)
- new net: J13.2 (Pin_2), M1.W7 (SWCLK)
- new net: J13.4 (Pin_4), M1.W6 (SWDIO)
- new net: J13.5 (Pin_5), M1.W5 (nReset)
- new net: M1.W2 (CAN_VIO), M4.V2 (CAN_VIO)
- new net: M1.W4 (CAN_TX), M4.V5 (CAN_TX)
- new net: M1.W3 (CAN_RX), M4.V6 (CAN_RX)
- new net: J7.3 (Pin_3), M1.E1 (LSU_Un)
- new net: J7.4 (Pin_4), M1.E2 (LSU_Vm)
- new net: J7.5 (Pin_5), M1.E3 (LSU_Ip)
- new net: J7.6 (Pin_6), M1.E4 (LSU_Rtrim)
- new net: J7.7 (Pin_7), J7.8 (Pin_8), M1.E5 (LSU_H+)
- new net: M1.J2 (SEL2), M1.J_VCC2 (PULL_UP2)
- new net +5VA: M1.W1 (V5_IN), M2.V1 (V5), M3.W1 (V5_IN), M4.V1 (V5)
- new net CAN_H: M2.S2 (CANH), M4.S2 (CANH)
- new net CAN_L: M2.S1 (CANL), M4.S1 (CANL)
- no-connect marks 10 -> 20
Other:
- note added: "#0"
- note added: "#1"

Commit message: трассировка
Connections:
- net CAN_H is gone; now on net CAN+: M2.S2 (CANH), M4.S2 (CANH)
- net CAN_L is gone; now on net CAN-: M2.S1 (CANL), M4.S1 (CANL)
- net 12V_MR: now also BRD1.B18(21) (12V_IGN)
Changed lines of the file:
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@@
     (effects (font (size 1.27 1.27)) (justify left bottom))
-  )
-  (label "CAN_H" (at 163.83 325.12 180)
-    (effects (font (size 1.27 1.27)) (justify right bottom))
   )
   (label "IGN1" (at 74.93 142.24 0)
@@
     (effects (font (size 1.27 1.27)) (justify left bottom))
   )
-  (label "CAN_H" (at 162.56 372.11 180)
-    (effects (font (size 1.27 1.27)) (justify right bottom))
-  )
   (label "5V_SENSE_1" (at 184.0145 273.05 0)
     (effects (font (size 1.27 1.27)) (justify left bottom))
@@
     (effects (font (size 1.27 1.27)) (justify left bottom))
   )
+  (label "CAN-" (at 158.2748 322.58 0)
+    (effects (font (size 1.27 1.27)) (justify left bottom))
+  )
   (label "IGN9" (at 97.79 255.27 0)
     (effects (font (size 1.27 1.27)) (justify left bottom))
@@
     (effects (font (size 1.27 1.27)) (justify left bottom))
   )
+  (label "CAN+" (at 158.2748 325.12 0)
+    (effects (font (size 1.27 1.27)) (justify left bottom))
+  )
   (label "AV7" (at 74.93 147.32 0)
     (effects (font (size 1.27 1.27)) (justify left bottom))
@@
     (effects (font (size 1.27 1.27)) (justify left bottom))
   )
-  (label "CAN_L" (at 162.56 369.57 180)
-    (effects (font (size 1.27 1.27)) (justify right bottom))
-  )
   (label "CAN-" (at 43.18 280.67 0)
     (effects (font (size 1.27 1.27)) (justify left bottom))
@@
     (effects (font (size 1.27 1.27)) (justify left bottom))
   )
+  (label "CAN+" (at 157.48 372.11 0)
+    (effects (font (size 1.27 1.27)) (justify left bottom))
+  )
   (label "ETB1-" (at 185.42 173.99 0)
     (effects (font (size 1.27 1.27)) (justify left bottom))
@@
     (effects (font (size 1.27 1.27)) (justify left bottom))
   )
-  (label "CAN_L" (at 163.83 322.58 180)
-    (effects (font (size 1.27 1.27)) (justify right bottom))
-  )
   (label "AV3" (at 74.93 50.8 0)
     (effects (font (size 1.27 1.27)) (justify left bottom))
@@
     (effects (font (size 1.27 1.27)) (justify left bottom))
   )
+  (label "CAN-" (at 157.48 369.57 0)
+    (effects (font (size 1.27 1.27)) (justify left bottom))
+  )
   (label "AT4" (at 43.18 288.29 0)
     (effects (font (size 1.27 1.27)) (justify left bottom))
@@
     (effects (font (size 1.27 1.27)) (justify left bottom))
   )
+  (label "12V_MR" (at 185.42 201.93 0)
+    (effects (font (size 1.27 1.27)) (justify left bottom))
+  )
