File: 5.0mustangProteusPnP.kicad_pcb (KiCad board)
At the start: 2 copper layers, 139.7 x 149.6 mm, 13 parts, among them J1 5-146280-3, J10 XH-10AW, J13 Conn_01x06, J2 5103308-3, J3 Conn_01x06, J4 5103308-3, J7 XH-10AW, M1 Module-wbo-0.3, M2 Module-can-0.1, M3 Module-wbo-0.3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

Commit message: new gerbers
Parts:
- moved BRD1 244.5 mm to (22.3, -70.0)
- moved J1 244.5 mm to (146.4, -154.9)
- moved J10 244.5 mm to (148.1, -31.4)
- moved J13 244.5 mm to (65.6, -53.1)
- moved J2 244.5 mm to (100.1, -63.2)
- moved J3 244.5 mm to (115.5, -31.7)
- moved J4 244.5 mm to (61.9, -63.2)
- moved J7 244.5 mm to (31.6, -53.9)
- moved M1 244.5 mm to (80.0, -49.7)
- moved M2 244.5 mm to (91.3, -47.9)
- moved M3 244.5 mm to (100.6, -34.8)
- moved M4 244.5 mm to (89.0, -36.5)
- moved U1 244.5 mm to (41.3, -160.3)
